Commit message: changed urdf file as per ROS2 humble requirements

File: urdf/robot_cell_controlled.urdf.xacro (robot description, xacro)
@@ -17,5 +17,8 @@
     <xacro:arg name="ur_input_recipe_filename" default="$(find ur_robot_driver)/resources/rtde_input_recipe.txt"/>
     <xacro:arg name="use_fake_hardware" default="false" />
-    <xacro:arg name="mock_sensor_commands" default="false" />
+    <xacro:arg name="fake_sensor_commands" default="false" />
+    <!--find hash_kinematics in kinematics_params-->
+    <xacro:property name="kinematics_params_file" value="$(arg kinematics_params)"/>
+    <xacro:property name="kinematics_hash" value="${xacro.load_yaml(kinematics_params_file)['kinematics']['hash']}"/>
     <link name="world"/>
     <!-- This will create the scene where the robot is located in -->
@@ -30,9 +33,9 @@
             <origin xyz="0 0 0" rpy="0 0 0"/>
     </xacro:robot_cell>
-    <!-- Create the control tag for the UR robot -->
+    <!--Create the control tag for the UR robot-->
     <xacro:ur_ros2_control
         name="$(arg ur_type)"
         tf_prefix="$(arg ur_type)_"
-        kinematics_parameters_file="$(arg kinematics_parameters_file)"
+        hash_kinematics="${kinematics_hash}"
         robot_ip="$(arg robot_ip)"
         script_filename="$(arg ur_script_filename)"
@@ -40,5 +43,5 @@
         input_recipe_filename="$(arg ur_input_recipe_filename)"
         use_fake_hardware="$(arg use_fake_hardware)"
-        mock_sensor_commands="$(arg mock_sensor_commands)"
+        fake_sensor_commands="$(arg fake_sensor_commands)"
         headless_mode="$(arg headless_mode)"
     />

Commit message: fixed kinematics parameters file name

File: urdf/robot_cell_controlled.urdf.xacro (robot description, xacro)
@@ -19,5 +19,5 @@
     <xacro:arg name="fake_sensor_commands" default="false" />
     <!--find hash_kinematics in kinematics_params-->
-    <xacro:property name="kinematics_params_file" value="$(arg kinematics_params)"/>
+    <xacro:property name="kinematics_params_file" value="$(arg kinematics_parameters_file)"/>
     <xacro:property name="kinematics_hash" value="${xacro.load_yaml(kinematics_params_file)['kinematics']['hash']}"/>
     <link name="world"/>

Commit message: updated urdf file

File: urdf/robot_cell_controlled.urdf.xacro (robot description, xacro)
@@ -7,8 +7,8 @@
     <!-- Specifying the arguments used for paprametrizing the description -->
     <xacro:arg name="ur_type" default="ur10e"/>
-    <xacro:arg name="joint_limits_parameters_file" default="$(find robot_cell_control)/config/$(arg ur_type)/joint_limits.yaml"/>
-    <xacro:arg name="kinematics_parameters_file" default="$(find robot_cell_control)/config/$(arg ur_type)/default_kinematics.yaml"/>
-    <xacro:arg name="physical_parameters_file" default="$(find robot_cell_control)/config/$(arg ur_type)/physical_parameters.yaml"/>
-    <xacro:arg name="visual_parameters_file" default="$(find robot_cell_control)/config/$(arg ur_type)/visual_parameters.yaml"/>
+    <xacro:arg name="joint_limit_params" default="$(find robot_cell_control)/config/$(arg ur_type)/joint_limits.yaml"/>
+    <xacro:arg name="kinematics_params" default="$(find robot_cell_control)/config/$(arg ur_type)/default_kinematics.yaml"/>
+    <xacro:arg name="physical_params" default="$(find robot_cell_control)/config/$(arg ur_type)/physical_parameters.yaml"/>
+    <xacro:arg name="visual_params" default="$(find robot_cell_control)/config/$(arg ur_type)/visual_parameters.yaml"/>
     <xacro:arg name="robot_ip" default="0.0.0.0"/>
     <xacro:arg name="headless_mode" default="false"/>
@@ -19,5 +19,5 @@
     <xacro:arg name="fake_sensor_commands" default="false" />
     <!--find hash_kinematics in kinematics_params-->
-    <xacro:property name="kinematics_params_file" value="$(arg kinematics_parameters_file)"/>
+    <xacro:property name="kinematics_params_file" value="$(arg kinematics_params)"/>
     <xacro:property name="kinematics_hash" value="${xacro.load_yaml(kinematics_params_file)['kinematics']['hash']}"/>
     <link name="world"/>
@@ -26,8 +26,8 @@
         parent="world"
         ur_type="$(arg ur_type)"
-        joint_limits_parameters_file="$(arg joint_limits_parameters_file)"
-        kinematics_parameters_file="$(arg kinematics_parameters_file)"
-        physical_parameters_file="$(arg physical_parameters_file)"
-        visual_parameters_file="$(arg visual_parameters_file)"
+        joint_limits_parameters_file="$(arg joint_limit_params)"
+        kinematics_parameters_file="$(arg kinematics_params)"
+        physical_parameters_file="$(arg physical_params)"
+        visual_parameters_file="$(arg visual_params)"
         >
             <origin xyz="0 0 0" rpy="0 0 0"/>
@@ -36,5 +36,5 @@
     <xacro:ur_ros2_control
         name="$(arg ur_type)"
-        tf_prefix="$(arg ur_type)_"
+        tf_prefix=""
         hash_kinematics="${kinematics_hash}"
         robot_ip="$(arg robot_ip)"
